File: board/ProtoPropDuo/ProtoPropDuo.kicad_pcb (KiCad board)
At the start: 2 copper layers, 98.8 x 72.3 mm, 354 parts, among them J1 Conn_01x04, J10 Conn_01x01, J100 Conn_01x01, J101 Conn_01x01, J102 Conn_01x01, J103 Conn_01x01, J104 Conn_01x01, J105 Conn_01x01, J106 Conn_01x01, J107 Conn_01x01, J108 Conn_01x01, J109 Conn_01x01, J11 Conn_01x01, J110 Conn_01x01, J111 Conn_01x01, J112 Conn_01x01, J113 Conn_01x01, J114 Conn_01x01, J115 Conn_01x01, J116 Conn_01x01, J117 Conn_01x01, J118 Conn_01x01, J12 Conn_01x01, J13 Conn_01x01, J14 Conn_01x01, J15 Conn_01x01, J16 Conn_01x01, J17 Conn_01x01, J18 Conn_01x01, J19 Conn_01x01, J2 Conn_01x07, J20 Conn_01x01, J21 Conn_01x01, J22 Conn_01x01, J23 Conn_01x01, J24 Conn_01x01, J25 Conn_01x01, J26 Conn_01x01, J27 Conn_01x01, J28 Conn_01x01, J29 Conn_01x01, J3 Conn_01x20, J30 Conn_01x01, J31 Conn_01x01, J32 Conn_01x01, J33 Conn_01x01, J34 Conn_01x01, J35 Conn_01x01, J36 Conn_01x01, J37 Conn_01x01, J38 Conn_01x01, J39 Conn_01x01, J4 Conn_01x20, J40 Conn_01x01, J41 Conn_01x01, J42 Conn_01x01, J43 Conn_01x01, J44 Conn_01x01, J45 Conn_01x01, J46 Conn_01x01, J47 Conn_01x01, J48 Conn_01x01, J49 Conn_01x01, J5 Conn_01x16, J50 Conn_01x01, J51 Conn_01x01, J52 Conn_01x01, J53 Conn_01x01, J54 Conn_01x01, J55 Conn_01x01, J56 Conn_01x01, J57 Conn_01x01, J58 Conn_01x01, J59 Conn_01x01, J6 Conn_01x12, J60 Conn_01x01, J61 Conn_01x01, J62 Conn_01x01, J63 Conn_01x01, J64 Conn_01x01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

Commit message: Rev B: Reworked the mapping from Pico to featherwing to align some pins for PIO and pwm channels. Added level shifter to support ws2812b individually addressable RGB lights and support for and external 5V power for servos on the extra Pico pins.
Parts:
- removed the REF** at (188.0, 106.7)
- removed the REF** at (223.5, 45.7)
- removed the REF** at (195.6, 101.6)
- removed the REF** at (210.8, 40.6)
- removed the REF** at (180.3, 58.4)
- removed the REF** at (193.0, 109.2)
- removed the REF** at (213.4, 45.7)
- removed the REF** at (218.4, 55.9)
- removed the REF** at (188.0, 109.2)
- removed the REF** at (218.4, 88.9)
- removed the REF** at (188.0, 96.5)
- removed the REF** at (213.4, 78.7)
- removed the REF** at (215.9, 86.4)
- removed the REF** at (177.8, 86.4)
- removed the REF** at (208.3, 81.3)
- removed the REF** at (195.6, 109.2)
- removed the REF** at (213.4, 71.1)
- removed the REF** at (218.4, 78.7)
- removed the REF** at (180.3, 45.7)
- removed the REF** at (215.9, 81.3)
- removed the REF** at (221.0, 45.7)
- removed the REF** at (182.9, 43.2)
- removed the REF** at (198.1, 109.2)
- removed the REF** at (198.1, 101.6)
- removed the REF** at (180.3, 96.5)
- removed the REF** at (218.4, 71.1)
- removed the REF** at (182.9, 81.3)
- removed the REF** at (193.0, 99.1)
- removed the REF** at (198.1, 99.1)
- removed the REF** at (193.0, 106.7)
- removed the REF** at (188.0, 81.3)
- removed the REF** at (180.3, 61.0)
- removed the REF** at (177.8, 76.2)
- removed the REF** at (193.0, 104.1)
- removed the REF** at (182.9, 83.8)
- removed the REF** at (177.8, 78.7)
- removed the REF** at (210.8, 68.6)
- removed the REF** at (188.0, 76.2)
- removed the REF** at (188.0, 99.1)
- removed the REF** at (188.0, 101.6)
- removed the REF** at (185.4, 104.1)
- removed the REF** at (180.3, 99.1)
- removed the REF** at (185.4, 88.9)
- removed the REF** at (210.8, 81.3)
- removed the REF** at (213.4, 61.0)
- removed the REF** at (188.0, 83.8)
- removed the REF** at (185.4, 96.5)
- removed the REF** at (208.3, 73.7)
- removed the REF** at (185.4, 81.3)
- removed the REF** at (185.4, 55.9)
- removed the REF** at (182.9, 106.7)
- removed the REF** at (215.9, 76.2)
- removed the REF** at (177.8, 63.5)
- removed the REF** at (213.4, 68.6)
- removed the REF** at (193.0, 101.6)
- removed the REF** at (208.3, 43.2)
- removed the REF** at (218.4, 40.6)
- removed the REF** at (210.8, 78.7)
- removed the REF** at (210.8, 76.2)
- removed the REF** at (218.4, 43.2)
- removed the REF** at (180.3, 86.4)
- removed the REF** at (215.9, 43.2)
- removed the REF** at (182.9, 45.7)
- removed the REF** at (213.4, 63.5)
- removed the REF** at (185.4, 101.6)
- removed the REF** at (182.9, 99.1)
- removed the REF** at (185.4, 83.8)
- removed the REF** at (218.4, 61.0)
- removed the REF** at (215.9, 78.7)
- removed the REF** at (188.0, 45.7)
- removed the REF** at (215.9, 68.6)
- removed the REF** at (177.8, 73.7)
- removed the REF** at (188.0, 78.7)
- removed the REF** at (188.0, 73.7)
- removed the REF** at (180.3, 73.7)
- removed the REF** at (208.3, 76.2)
- removed the REF** at (190.5, 101.6)
- removed the REF** at (195.6, 96.5)
- removed the REF** at (208.3, 45.7)
- removed the REF** at (188.0, 40.6)
- removed the REF** at (185.4, 71.1)
- removed the REF** at (213.4, 83.8)
- removed the REF** at (182.9, 58.4)
- removed the REF** at (208.3, 68.6)
- removed the REF** at (218.4, 81.3)
- removed the REF** at (190.5, 109.2)
- removed the REF** at (177.8, 43.2)
- removed the REF** at (195.6, 94.0)
- removed the REF** at (177.8, 81.3)
- removed the REF** at (208.3, 83.8)
- removed the REF** at (208.3, 58.4)
- removed the REF** at (185.4, 43.2)
- removed the REF** at (213.4, 73.7)
- removed the REF** at (210.8, 58.4)
- removed the REF** at (180.3, 78.7)
- removed the REF** at (182.9, 86.4)
- removed the REF** at (195.6, 106.7)
- removed the REF** at (213.4, 76.2)
- removed the REF** at (213.4, 40.6)
- removed the REF** at (208.3, 66.0)
- removed the REF** at (208.3, 71.1)
- removed the REF** at (213.4, 58.4)
- removed the REF** at (182.9, 76.2)
- removed the REF** at (182.9, 104.1)
- removed the REF** at (185.4, 61.0)
- removed the REF** at (215.9, 83.8)
- removed the REF** at (218.4, 58.4)
- removed the REF** at (213.4, 66.0)
- removed the REF** at (185.4, 73.7)
- removed the REF** at (210.8, 86.4)
- removed the REF** at (210.8, 55.9)
- removed the REF** at (218.4, 68.6)
- removed the REF** at (188.0, 86.4)
- removed the REF** at (188.0, 43.2)
- removed the REF** at (182.9, 55.9)
- removed the REF** at (182.9, 68.6)
- removed the REF** at (182.9, 88.9)
- removed the REF** at (215.9, 63.5)
- removed the REF** at (210.8, 45.7)
- removed the REF** at (215.9, 88.9)
- removed the REF** at (185.4, 45.7)
- removed the REF** at (188.0, 66.0)
- removed the REF** at (188.0, 94.0)
- removed the REF** at (218.4, 83.8)
- removed the REF** at (182.9, 66.0)
- removed the REF** at (182.9, 96.5)
- removed the REF** at (180.3, 66.0)
- removed the REF** at (210.8, 66.0)
- removed the REF** at (182.9, 73.7)
- removed the REF** at (177.8, 58.4)
- removed the REF** at (213.4, 81.3)
- removed the REF** at (185.4, 40.6)
- removed the REF** at (188.0, 88.9)
- removed the REF** at (177.8, 55.9)
- removed the REF** at (190.5, 96.5)
- removed the REF** at (215.9, 40.6)
- removed the REF** at (188.0, 58.4)
- removed the REF** at (195.6, 99.1)
- removed the REF** at (185.4, 76.2)
- removed the REF** at (213.4, 55.9)
- removed the REF** at (188.0, 71.1)
- removed the REF** at (180.3, 101.6)
- removed the REF** at (188.0, 61.0)
- removed the REF** at (208.3, 40.6)
- removed the REF** at (185.4, 78.7)
- removed the REF** at (190.5, 104.1)
- removed the REF** at (218.4, 45.7)
- removed the REF** at (198.1, 96.5)
- removed the REF** at (198.1, 94.0)
- removed the REF** at (213.4, 86.4)
- removed the REF** at (195.6, 104.1)
- removed the REF** at (185.4, 58.4)
- removed the REF** at (218.4, 86.4)
- removed the REF** at (180.3, 71.1)
- removed the REF** at (188.0, 63.5)
- removed the REF** at (210.8, 88.9)
- removed the REF** at (210.8, 63.5)
- removed the REF** at (198.1, 106.7)
- removed the REF** at (185.4, 106.7)
- removed the REF** at (177.8, 61.0)
- removed the REF** at (180.3, 63.5)
- removed the REF** at (185.4, 99.1)
- removed the REF** at (218.4, 76.2)
- removed the REF** at (218.4, 63.5)
- removed the REF** at (180.3, 109.2)
- removed the REF** at (180.3, 76.2)
- removed the REF** at (180.3, 40.6)
- removed the REF** at (193.0, 96.5)
- removed the REF** at (215.9, 61.0)
- removed the REF** at (180.3, 88.9)
- removed the REF** at (193.0, 94.0)
- removed the REF** at (185.4, 109.2)
- removed the REF** at (185.4, 63.5)
- removed the REF** at (210.8, 83.8)
- removed the REF** at (180.3, 68.6)
- removed the REF** at (190.5, 99.1)
- removed the REF** at (185.4, 86.4)
- removed the REF** at (210.8, 71.1)
- removed the REF** at (215.9, 45.7)
- removed the REF** at (182.9, 40.6)
- removed the REF** at (208.3, 86.4)
- removed the REF** at (185.4, 94.0)
- removed the REF** at (208.3, 61.0)
- removed the REF** at (215.9, 71.1)
- removed the REF** at (177.8, 83.8)
- removed the REF** at (215.9, 73.7)
- removed the REF** at (182.9, 61.0)
- removed the REF** at (208.3, 55.9)
- removed the REF** at (182.9, 94.0)
- removed the REF** at (182.9, 78.7)
- removed the REF** at (177.8, 40.6)
- removed the REF** at (188.0, 68.6)
- removed the REF** at (182.9, 71.1)
- removed the REF** at (180.3, 83.8)
- removed the REF** at (177.8, 45.7)
- removed the REF** at (177.8, 71.1)
- removed the REF** at (208.3, 63.5)
- removed the REF** at (180.3, 94.0)
- removed the REF** at (215.9, 55.9)
- removed the REF** at (213.4, 88.9)
- removed the REF** at (180.3, 81.3)
- removed the REF** at (180.3, 104.1)
- removed the REF** at (215.9, 66.0)
- removed the REF** at (208.3, 78.7)
- removed the REF** at (210.8, 73.7)
- removed the REF** at (185.4, 68.6)
- removed the REF** at (177.8, 68.6)
- removed the REF** at (208.3, 88.9)
- removed the REF** at (210.8, 43.2)
- removed the REF** at (210.8, 61.0)
- removed the REF** at (182.9, 101.6)
- removed the REF** at (188.0, 104.1)
- removed the REF** at (215.9, 58.4)
- removed the REF** at (177.8, 66.0)
- removed the REF** at (218.4, 73.7)
- removed the REF** at (180.3, 55.9)
- removed the REF** at (185.4, 66.0)
- removed the REF** at (190.5, 94.0)
- removed the REF** at (177.8, 88.9)
- removed the REF** at (213.4, 43.2)
- removed the REF** at (218.4, 66.0)
- removed the REF** at (180.3, 106.7)
- removed the REF** at (198.1, 104.1)
- removed the REF** at (182.9, 63.5)
- removed the REF** at (188.0, 55.9)
- removed the REF** at (180.3, 43.2)
- removed the REF** at (190.5, 106.7)
- removed the REF** at (182.9, 109.2)
- added ?: , , F.Cu at (210.8, 86.4)
- added ?: , , F.Cu at (208.3, 83.8)
- added ?: , , F.Cu at (213.4, 61.0)
- added ?: , , F.Cu at (182.9, 58.4)
- added ?: , , F.Cu at (180.3, 40.6)
- added ?: , , F.Cu at (185.4, 45.7)
- added ?: , , F.Cu at (215.9, 71.1)
- added ?: , , F.Cu at (215.9, 81.3)
- added ?: , , F.Cu at (182.9, 55.9)
- added ?: , , F.Cu at (208.3, 78.7)
- added ?: , , F.Cu at (218.4, 76.2)
- added ?: , , F.Cu at (177.8, 40.6)
- added ?: , , F.Cu at (213.4, 88.9)
- added ?: , , F.Cu at (185.4, 66.0)
- added ?: , , F.Cu at (182.9, 76.2)
- added ?: , , F.Cu at (210.8, 55.9)
- added ?: , , F.Cu at (213.4, 43.2)
- added ?: , , F.Cu at (182.9, 40.6)
- added ?: , , F.Cu at (210.8, 58.4)
- added ?: , , F.Cu at (213.4, 83.8)
- added ?: , , F.Cu at (210.8, 61.0)
- added ?: , , F.Cu at (185.4, 40.6)
- added ?: , , F.Cu at (185.4, 55.9)
- added ?: , , F.Cu at (210.8, 45.7)
- added ?: , , F.Cu at (185.4, 68.6)
- added ?: , , F.Cu at (188.0, 76.2)
- added ?: , , F.Cu at (213.4, 86.4)
- added ?: , , F.Cu at (210.8, 73.7)
- added ?: , , F.Cu at (210.8, 78.7)
- added ?: , , F.Cu at (218.4, 45.7)
- added ?: , , F.Cu at (185.4, 71.1)
- added ?: , , F.Cu at (208.3, 68.6)
- added ?: , , F.Cu at (177.8, 88.9)
- added ?: , , F.Cu at (177.8, 66.0)
- added ?: , , F.Cu at (218.4, 43.2)
- added ?: , , F.Cu at (218.4, 88.9)
- added ?: , , F.Cu at (180.3, 71.1)
- added ?: , , F.Cu at (177.8, 58.4)
- added ?: , , F.Cu at (190.5, 45.7)
- added ?: , , F.Cu at (213.4, 66.0)
- added ?: , , F.Cu at (188.0, 71.1)
- added ?: , , F.Cu at (208.3, 40.6)
- added ?: , , F.Cu at (215.9, 66.0)
- added ?: , , F.Cu at (210.8, 81.3)
- added ?: , , F.Cu at (180.3, 58.4)
- added ?: , , F.Cu at (210.8, 68.6)
- added ?: , , F.Cu at (177.8, 86.4)
- added ?: , , F.Cu at (213.4, 63.5)
- added ?: , , F.Cu at (182.9, 68.6)
- added ?: , , F.Cu at (215.9, 83.8)
- added ?: , , F.Cu at (182.9, 78.7)
- added ?: , , F.Cu at (180.3, 78.7)
- added ?: , , F.Cu at (208.3, 45.7)
- added ?: , , F.Cu at (215.9, 58.4)
- added ?: , , F.Cu at (218.4, 63.5)
- added ?: , , F.Cu at (185.4, 61.0)
- added ?: , , F.Cu at (188.0, 81.3)
- added ?: , , F.Cu at (185.4, 109.2)
- added ?: , , F.Cu at (215.9, 86.4)
- added ?: , , F.Cu at (218.4, 68.6)
- added ?: , , F.Cu at (215.9, 45.7)
- added ?: , , F.Cu at (215.9, 88.9)
- added ?: , , F.Cu at (210.8, 88.9)
- added ?: , , F.Cu at (185.4, 58.4)
- added ?: , , F.Cu at (215.9, 73.7)
- added ?: , , F.Cu at (177.8, 78.7)
- added ?: , , F.Cu at (188.0, 83.8)
- added ?: , , F.Cu at (188.0, 66.0)
- added ?: , , F.Cu at (180.3, 55.9)
- added ?: , , F.Cu at (208.3, 58.4)
- added ?: , , F.Cu at (177.8, 43.2)
- added ?: , , F.Cu at (180.3, 83.8)
- added ?: , , F.Cu at (210.8, 40.6)
- added ?: , , F.Cu at (208.3, 73.7)
- added ?: , , F.Cu at (215.9, 43.2)
- added ?: , , F.Cu at (188.0, 61.0)
- added ?: , , F.Cu at (215.9, 55.9)
- added ?: , , F.Cu at (182.9, 43.2)
- added ?: , , F.Cu at (210.8, 63.5)
- added ?: , , F.Cu at (182.9, 71.1)
- added ?: , , F.Cu at (185.4, 88.9)
- added ?: , , F.Cu at (177.8, 73.7)
- added ?: , , F.Cu at (182.9, 61.0)
- added ?: , , F.Cu at (180.3, 88.9)
- added ?: , , F.Cu at (182.9, 83.8)
- added ?: , , F.Cu at (182.9, 88.9)
- added ?: , , F.Cu at (185.4, 73.7)
- added ?: , , F.Cu at (185.4, 81.3)
- added ?: , , F.Cu at (177.8, 63.5)
- added ?: , , F.Cu at (185.4, 83.8)
- added ?: , , F.Cu at (188.0, 86.4)
- added ?: , , F.Cu at (218.4, 86.4)
- added ?: , , F.Cu at (218.4, 66.0)
- added ?: , , F.Cu at (177.8, 68.6)
- added ?: , , F.Cu at (177.8, 45.7)
- added ?: , , F.Cu at (213.4, 81.3)
- added ?: , , F.Cu at (208.3, 55.9)
- added ?: , , F.Cu at (180.3, 73.7)
- added ?: , , F.Cu at (218.4, 71.1)
- added ?: , , F.Cu at (188.0, 45.7)
- added ?: , , F.Cu at (208.3, 71.1)
- added ?: , , F.Cu at (218.4, 40.6)
- added ?: , , F.Cu at (177.8, 76.2)
- added ?: , , F.Cu at (213.4, 40.6)
- added ?: , , F.Cu at (182.9, 86.4)
- added ?: , , F.Cu at (215.9, 61.0)
- added ?: , , F.Cu at (218.4, 73.7)
- added ?: , , F.Cu at (177.8, 81.3)
- added ?: , , F.Cu at (210.8, 43.2)
- added ?: , , F.Cu at (218.4, 83.8)
- added ?: , , F.Cu at (182.9, 81.3)
- added ?: , , F.Cu at (215.9, 40.6)
- added ?: , , F.Cu at (208.3, 61.0)
- added ?: , , F.Cu at (208.3, 76.2)
- added ?: , , F.Cu at (213.4, 71.1)
- added ?: , , F.Cu at (208.3, 81.3)
- added ?: , , F.Cu at (215.9, 76.2)
- added ?: , , F.Cu at (208.3, 63.5)
- added ?: , , F.Cu at (180.3, 63.5)
- added ?: , , F.Cu at (208.3, 86.4)
- added ?: , , F.Cu at (188.0, 55.9)
- added ?: , , F.Cu at (223.5, 45.7)
- added ?: , , F.Cu at (185.4, 86.4)
- added ?: , , F.Cu at (213.4, 68.6)
- added ?: , , F.Cu at (215.9, 68.6)
- added ?: , , F.Cu at (182.9, 73.7)
- added ?: , , F.Cu at (210.8, 66.0)
- added ?: , , F.Cu at (188.0, 40.6)
- added ?: , , F.Cu at (208.3, 66.0)
- added ?: , , F.Cu at (218.4, 61.0)
- added ?: , , F.Cu at (180.3, 76.2)
- added ?: , , F.Cu at (208.3, 43.2)
- added ?: , , F.Cu at (218.4, 55.9)
- added ?: , , F.Cu at (188.0, 58.4)
- added ?: , , F.Cu at (213.4, 76.2)
- added ?: , , F.Cu at (213.4, 45.7)
- added ?: , , F.Cu at (188.0, 88.9)
- added ?: , , F.Cu at (180.3, 66.0)
- added ?: , , F.Cu at (210.8, 83.8)
- added ?: , , F.Cu at (215.9, 78.7)
- added ?: , , F.Cu at (221.0, 45.7)
- added ?: , , F.Cu at (218.4, 81.3)
- added ?: , , F.Cu at (182.9, 45.7)
- added ?: , , F.Cu at (180.3, 81.3)
- added ?: , , F.Cu at (193.0, 45.7)
- added ?: , , F.Cu at (213.4, 73.7)
- added ?: , , F.Cu at (180.3, 86.4)
- added ?: , , F.Cu at (215.9, 63.5)
- added ?: , , F.Cu at (185.4, 43.2)
- added ?: , , F.Cu at (177.8, 61.0)
- added ?: , , F.Cu at (177.8, 83.8)
- added ?: , , F.Cu at (188.0, 68.6)
- added ?: , , F.Cu at (208.3, 88.9)
- added ?: , , F.Cu at (218.4, 58.4)
- added ?: , , F.Cu at (180.3, 45.7)
- added ?: , , F.Cu at (180.3, 61.0)
- added ?: , , F.Cu at (213.4, 55.9)
- added ?: , , F.Cu at (180.3, 43.2)
- added ?: , , F.Cu at (218.4, 78.7)
- added ?: , , F.Cu at (213.4, 58.4)
- added ?: , , F.Cu at (177.8, 71.1)
- added ?: , , F.Cu at (185.4, 63.5)
- added ?: , , F.Cu at (188.0, 78.7)
- added ?: , , F.Cu at (188.0, 43.2)
- added ?: , , F.Cu at (210.8, 71.1)
- added ?: , , F.Cu at (185.4, 78.7)
- added ?: , , F.Cu at (210.8, 76.2)
- added ?: , , F.Cu at (185.4, 76.2)
- added ?: , , F.Cu at (180.3, 68.6)
- added ?: , , F.Cu at (188.0, 73.7)
- added ?: , , F.Cu at (182.9, 66.0)
- added ?: , , F.Cu at (188.0, 63.5)
- added ?: , , F.Cu at (182.9, 63.5)
- added ?: , , F.Cu at (213.4, 78.7)
- added C1: 0.1uF, Capacitor_SMD:C_0603_1608Metric_Pad1.08x0.95mm_HandSolder, F.Cu at (204.5, 99.1)
- added J110: Conn_01x01, Department of Alchemy:Grid Hole, F.Cu at (182.9, 99.1)
- added J110: Conn_01x01, Department of Alchemy:Grid Hole, F.Cu at (188.0, 99.1)
- added J110: Conn_01x01, Department of Alchemy:Grid Hole, F.Cu at (190.5, 99.1)
- added J110: Conn_01x01, Department of Alchemy:Grid Hole, F.Cu at (185.4, 99.1)
- added J110: Conn_01x01, Department of Alchemy:Grid Hole, F.Cu at (193.0, 99.1)
- added J110: Conn_01x01, Department of Alchemy:Grid Hole, F.Cu at (180.3, 99.1)
- added J113: Conn_01x01, Department of Alchemy:Grid Hole, F.Cu at (188.0, 109.2)
- added J113: Conn_01x01, Department of Alchemy:Grid Hole, F.Cu at (180.3, 109.2)
- added J113: Conn_01x01, Department of Alchemy:Grid Hole, F.Cu at (193.0, 109.2)
- added J113: Conn_01x01, Department of Alchemy:Grid Hole, F.Cu at (182.9, 109.2)
- added J113: Conn_01x01, Department of Alchemy:Grid Hole, F.Cu at (190.5, 109.2)
- added J114: Conn_01x01, Department of Alchemy:Grid Hole, F.Cu at (188.0, 106.7)
- added J114: Conn_01x01, Department of Alchemy:Grid Hole, F.Cu at (190.5, 106.7)
- added J114: Conn_01x01, Department of Alchemy:Grid Hole, F.Cu at (180.3, 106.7)
- added J114: Conn_01x01, Department of Alchemy:Grid Hole, F.Cu at (185.4, 106.7)
- added J114: Conn_01x01, Department of Alchemy:Grid Hole, F.Cu at (193.0, 106.7)
- added J114: Conn_01x01, Department of Alchemy:Grid Hole, F.Cu at (182.9, 106.7)
- added J115: Conn_01x01, Department of Alchemy:Grid Hole, F.Cu at (180.3, 104.1)
- added J115: Conn_01x01, Department of Alchemy:Grid Hole, F.Cu at (188.0, 104.1)
- added J115: Conn_01x01, Department of Alchemy:Grid Hole, F.Cu at (182.9, 104.1)
- added J115: Conn_01x01, Department of Alchemy:Grid Hole, F.Cu at (185.4, 104.1)
- added J115: Conn_01x01, Department of Alchemy:Grid Hole, F.Cu at (193.0, 104.1)
- added J115: Conn_01x01, Department of Alchemy:Grid Hole, F.Cu at (190.5, 104.1)
- added J116: Conn_01x01, Department of Alchemy:Grid Hole, F.Cu at (190.5, 101.6)
- added J116: Conn_01x01, Department of Alchemy:Grid Hole, F.Cu at (182.9, 101.6)
- added J116: Conn_01x01, Department of Alchemy:Grid Hole, F.Cu at (188.0, 101.6)
- added J116: Conn_01x01, Department of Alchemy:Grid Hole, F.Cu at (180.3, 101.6)
- added J116: Conn_01x01, Department of Alchemy:Grid Hole, F.Cu at (193.0, 101.6)
- added J116: Conn_01x01, Department of Alchemy:Grid Hole, F.Cu at (185.4, 101.6)
- added J118: Conn_01x01, Department of Alchemy:Grid Hole, F.Cu at (180.3, 96.5)
- added J118: Conn_01x01, Department of Alchemy:Grid Hole, F.Cu at (188.0, 96.5)
- added J118: Conn_01x01, Department of Alchemy:Grid Hole, F.Cu at (193.0, 96.5)
- added J118: Conn_01x01, Department of Alchemy:Grid Hole, F.Cu at (190.5, 96.5)
- added J118: Conn_01x01, Department of Alchemy:Grid Hole, F.Cu at (182.9, 96.5)
- added J118: Conn_01x01, Department of Alchemy:Grid Hole, F.Cu at (185.4, 96.5)
- added J119: Conn_01x01, Department of Alchemy:Grid Hole, F.Cu at (175.3, 94.0)
- added J120: Conn_01x01, Department of Alchemy:Grid Hole, F.Cu at (180.3, 94.0)
- added J120: Conn_01x01, Department of Alchemy:Grid Hole, F.Cu at (182.9, 94.0)
- added J120: Conn_01x01, Department of Alchemy:Grid Hole, F.Cu at (190.5, 94.0)
- added J120: Conn_01x01, Department of Alchemy:Grid Hole, F.Cu at (177.8, 94.0)
- added J120: Conn_01x01, Department of Alchemy:Grid Hole, F.Cu at (188.0, 94.0)
- added J120: Conn_01x01, Department of Alchemy:Grid Hole, F.Cu at (185.4, 94.0)
- added J120: Conn_01x01, Department of Alchemy:Grid Hole, F.Cu at (193.0, 94.0)
- added J121: Conn_01x03, Connector_PinHeader_2.54mm:PinHeader_1x03_P2.54mm_Vertical, F.Cu at (143.3, 96.0)
- added J122: Conn_01x02, Connector_PinHeader_2.54mm:PinHeader_1x02_P2.54mm_Vertical, F.Cu at (228.6, 96.5)
- added J123: Conn_01x05_Extra_Output, Connector_PinHeader_2.54mm:PinHeader_1x05_P2.54mm_Vertical, F.Cu at (218.4, 99.1)
- added J124: Conn_01x05, Connector_PinHeader_2.54mm:PinHeader_1x05_P2.54mm_Vertical, F.Cu at (215.9, 99.1)
- added JP1: SolderJumper_2_Bridged, Jumper:SolderJumper-2_P1.3mm_Bridged_Pad1.0x1.5mm, B.Cu at (222.9, 94.7)
- added JP2: SolderJumper_3_Bridged12, Jumper:SolderJumper-3_P1.3mm_Bridged12_Pad1.0x1.5mm, B.Cu at (201.9, 92.8)
- added JP3: SolderJumper_3_Bridged12, Jumper:SolderJumper-3_P1.3mm_Bridged12_Pad1.0x1.5mm, B.Cu at (201.9, 98.0)
- added R1: 300, Resistor_SMD:R_0603_1608Metric_Pad0.98x0.95mm_HandSolder, F.Cu at (210.4, 99.2)
- added R2: 300, Resistor_SMD:R_0603_1608Metric_Pad0.98x0.95mm_HandSolder, F.Cu at (210.4, 101.7)
- added R3: 300, Resistor_SMD:R_0603_1608Metric_Pad0.98x0.95mm_HandSolder, F.Cu at (210.4, 104.2)
- added R4: 300, Resistor_SMD:R_0603_1608Metric_Pad0.98x0.95mm_HandSolder, F.Cu at (210.4, 106.7)
- added R5: 300, Resistor_SMD:R_0603_1608Metric_Pad0.98x0.95mm_HandSolder, F.Cu at (210.4, 109.2)
- added REF**: PinHeader_1x01_P2.54mm_Vertical, Connector_PinHeader_2.54mm:PinHeader_1x01_P2.54mm_Vertical, F.Cu at (177.8, 55.9)
- added U2: ~, Department of Alchemy:SOP65P640X120-20N, F.Cu at (201.9, 104.1)
- J106, J112: value Conn_01x01 -> Conn_01x05; footprint Department of Alchemy:Grid Hole -> Connector_PinHeader_2.54mm:PinHeader_1x05_P2.54mm_Vertical
- moved J106 46.8 mm to (221.0, 99.1)
- moved J112 46.8 mm to (223.5, 99.1)
- moved J110 3.59 mm to (177.8, 99.1)
- moved J117 3.59 mm to (175.3, 99.1)
- moved J107 2.54 mm to (175.3, 106.7)
- moved J108 2.54 mm to (175.3, 104.1)
- moved J114 2.54 mm to (177.8, 106.7)
- moved J115 2.54 mm to (177.8, 104.1)
- moved J109 2.54 mm to (175.3, 101.6)
- moved J111 2.54 mm to (175.3, 96.5)
- moved J113 2.54 mm to (177.8, 109.2)
- moved J116 2.54 mm to (177.8, 101.6)
- moved J118 2.54 mm to (177.8, 96.5)
- moved J7 2.54 mm to (175.3, 109.2)
Connections:
- J106 pad 1: /GPIO19 -> +5V
- J107 pad 1: /GPIO17 -> /GPIO21
- J108 pad 1: /GPIO16 -> /GPIO20
- J109 pad 1: /GPIO7 -> /GPIO19
- J110 pad 1: /VSYS -> /GPIO18
- J111 pad 1: /AGND -> /VSYS
- J112 pad 1: /GPIO19 -> GND
- J113 pad 1: /GPIO18 -> /GPIO22
- J114 pad 1: /GPIO17 -> /GPIO21
- J115 pad 1: /GPIO16 -> /GPIO20
- J116 pad 1: /GPIO7 -> /GPIO19
- J117 pad 1: /VSYS -> /GPIO18
- J118 pad 1: /AGND -> /VSYS
- J2 pad 3: /GPIO7 -> /GPIO18
- J2 pad 4: /GPIO16 -> /GPIO19
- J2 pad 5: /GPIO17 -> /GPIO20
- J2 pad 6: /GPIO18 -> /GPIO21
- J2 pad 7: /GPIO19 -> /GPIO22
- J3 pad 10: /GPIO7 -> /D5
- J3 pad 12: /D9 -> /D6
- J3 pad 14: /D10 -> /D9
- J3 pad 15: /D11 -> /D10
- J3 pad 16: /D12 -> /D4
- J3 pad 17: /D13 -> /D11
- J3 pad 6: /D4 -> /A3
- J3 pad 7: /D5 -> /D24
- J3 pad 9: /D6 -> /D25
- J4 pad 1: /GPIO16 -> /D12
- J4 pad 2: /GPIO17 -> /D13
- J4 pad 6: /A3 -> /GPIO20
- J4 pad 7: /D24 -> /GPIO21
- J4 pad 9: /D25 -> /GPIO22
- J7 pad 1: /GPIO18 -> /GPIO22
- U1 pad 10: /GPIO7 -> /D5
- U1 pad 12: /D9 -> /D6
- U1 pad 14: /D10 -> /D9
- U1 pad 15: /D11 -> /D10
- U1 pad 16: /D12 -> /D4
- U1 pad 17: /D13 -> /D11
- U1 pad 21: /GPIO16 -> /D12
- U1 pad 22: /GPIO17 -> /D13
- U1 pad 26: /A3 -> /GPIO20
- U1 pad 27: /D24 -> /GPIO21
- U1 pad 29: /D25 -> /GPIO22
- U1 pad 41: unconnected-(U1-SWCLK-Pad41) -> /SWCLK
- U1 pad 42: unconnected-(U1-GND-Pad42) -> GND
- U1 pad 43: unconnected-(U1-SWDIO-Pad43) -> /SWDIO
- U1 pad 6: /D4 -> /A3
- U1 pad 7: /D5 -> /D24
- U1 pad 9: /D6 -> /D25
Routing:
- net /GPIO22: track 0.00 -> 92.5 mm, vias 0 -> 3
- net /GPIO7: track 83.7 -> 0.00 mm, vias 1 -> 0
- net /GPIO21: track 0.00 -> 82.2 mm, vias 0 -> 3
- net +3.3V: track 155.1 -> 229.5 mm
- net /GPIO20: track 0.00 -> 67.1 mm, vias 0 -> 5
- net /VBUS: track 85.7 -> 140.8 mm
- net /GPIO17: track 40.1 -> 0.00 mm, vias 1 -> 0
- net /GPIO16: track 34.5 -> 0.00 mm, vias 1 -> 0
- net /D25: track 44.9 -> 70.2 mm
- net /D13: track 105.9 -> 81.4 mm
- net /D24: track 49.6 -> 73.6 mm
- net GND: track 143.8 -> 120.4 mm, vias 16 -> 21
- net +5V: track 0.00 -> 21.3 mm
- net /D12: track 102.9 -> 82.3 mm
- net /A3: track 54.3 -> 74.3 mm, vias 2 -> 0
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Other:
- board text added: "+5"
- board text added: "3"
- board text added: "B"
- board text added: "DATA"
- board text added: "DEBUG"
- board text added: "EXTERNAL"
- board text added: "EXTERNAL POWER"
- board text added: "GP16 /12"
- board text added: "GP17 /13"
- board text added: "GP20"
- board text added: "GP21"
- board text added: "GP22"
- board text added: "GPIO20"
- board text added: "GPIO21"
- board text added: "GPIO22"
- board text added: "IN"
- board text added: "OUT"
- board text added: "Proto Prop Duo"
- board text added: "SERVO"
- board text added: "WS2812B"
- board text removed: "GP16"
- board text removed: "GP17"
- board text removed: "GP20/A3"
- board text removed: "GP21/24"
- board text removed: "GP22/25"
- board text removed: "GPIO16"
- board text removed: "GPIO17"
- board text removed: "GPIO7"
- board text removed: "Raspberry Pi Pico FeatherWing Duo"
- board text removed: "Rev 1"
